Commit message: push fixed cordinate joint 2

File: CADModel/AssemblyDraft1/urdf/AssemblyDraft1.urdf (robot description, URDF)
Before this commit: robot RobotAssembly, 8 links, 7 joints
Links:
- link BaseLink: geometry collision mesh filename=package://AssemblyDraft1/meshes/BaseLink.STL; visual mesh filename=package://AssemblyDraft1/meshes/BaseLink.STL
- link J1_Link: geometry collision mesh filename=package://AssemblyDraft1/meshes/J1_Link.STL; visual mesh filename=package://AssemblyDraft1/meshes/J1_Link.STL
- link J2_Link: geometry collision mesh filename=package://AssemblyDraft1/meshes/J2_Link.STL; visual mesh filename=package://AssemblyDraft1/meshes/J2_Link.STL
- link J3_Link: geometry collision mesh filename=package://AssemblyDraft1/meshes/J3_Link.STL; visual mesh filename=package://AssemblyDraft1/meshes/J3_Link.STL
- link J4_Link: geometry collision mesh filename=package://AssemblyDraft1/meshes/J4_Link.STL; visual mesh filename=package://AssemblyDraft1/meshes/J4_Link.STL
- link J5_Link: geometry collision mesh filename=package://AssemblyDraft1/meshes/J5_Link.STL; visual mesh filename=package://AssemblyDraft1/meshes/J5_Link.STL
- link J6_Link: geometry collision mesh filename=package://AssemblyDraft1/meshes/J6_Link.STL; visual mesh filename=package://AssemblyDraft1/meshes/J6_Link.STL
- link base_Frame: geometry collision mesh filename=package://AssemblyDraft1/meshes/base_Frame.STL; visual mesh filename=package://AssemblyDraft1/meshes/base_Frame.STL
Joints:
- joint J1: limit lower=-6.2856 upper=6.2856 effort=0 velocity=0 -> lower=-6.2856 upper=6.2856 effort=5 velocity=5
- joint J2: limit lower=-6.2856 upper=6.2856 effort=0 velocity=0 -> lower=-6.2856 upper=6.2856 effort=5 velocity=5; origin xyz=0 0 0.0450235133971798 rpy=1.5707963267949 -1.57001254680866 -3.14159265358979 -> xyz=0 0 0.045024 rpy=1.5708 -1.57 -3.1416
- joint J3: limit lower=-6.2856 upper=6.2856 effort=0 velocity=0 -> lower=-6.2856 upper=6.2856 effort=5 velocity=5; origin xyz=0.0999764866100428 0 0.035 rpy=0 0 1.57158010678112 -> xyz=0.099976 0 0.035 rpy=0 0 1.5716
- joint J4: limit lower=-6.2856 upper=6.2856 effort=0 velocity=0 -> lower=-6.2856 upper=6.2856 effort=5 velocity=5; origin xyz=0.0399655013979157 -0.0440313376813969 -0.0344999999999999 rpy=1.5707963267949 0 1.57001254680867 -> xyz=0.039966 -0.044031 -0.0345 rpy=1.5708 0 1.57
- joint J5: limit lower=-6.2856 upper=6.2856 effort=0 velocity=0 -> lower=-6.2856 upper=6.2856 effort=5 velocity=5; origin xyz=0 0.0345 0.0419999999999999 rpy=-1.5707963267949 0 0 -> xyz=0 0.0345 0.042 rpy=-1.5708 0 0
- joint J6: limit lower=-6.2856 upper=6.2856 effort=0 velocity=0 -> lower=-6.2856 upper=6.2856 effort=5 velocity=5
